File: pcb/cap-charger.kicad_sch (KiCad schematic)
At the start: 21 parts, among them U5 PTN04050CAZ, U6 LTC4425

Commit message: Replaced through-hole components with SMD
- Other small edits (e.g. optional jumper to force USB-boot)
Other:
- company: (none) -> Open Ephys, Inc.
- title: (none) -> Open Ephys Commutator Controller
Changed lines of the file:
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@@
 	(generator_version "8.0")
 	(paper "A4")
+	(title_block
+		(title "Open Ephys Commutator Controller")
+		(rev "D")
+		(company "Open Ephys, Inc.")
+	)
 	(junction
 		(at 86.36 93.98)
