File: pcb/motor-driver.kicad_sch (KiCad schematic)
At the start: 15 parts, among them J3 1719730004, U7 TMC2130-LA

Commit message: Replaced through-hole components with SMD
- Other small edits (e.g. optional jumper to force USB-boot)
Other:
- company: (none) -> Open Ephys, Inc.
- title: (none) -> Open Ephys Commutator Controller
Changed lines of the file:
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@@
 	(generator_version "8.0")
 	(paper "A4")
+	(title_block
+		(title "Open Ephys Commutator Controller")
+		(rev "D")
+		(company "Open Ephys, Inc.")
+	)
 	(junction
 		(at 176.53 44.45)

Commit message: Add GPIO to programming header
Parts:
- J3: footprint open-ephys:MOLEX_1719730004_1x04_P2.54mm_Vert_Lock -> oe:MOLEX_1719730004_1x04_P2.54mm_Vert_Lock
Changed lines of the file:
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@@
 			)
 		)
-		(property "Footprint" "open-ephys:MOLEX_1719730004_1x04_P2.54mm_Vert_Lock"
+		(property "Footprint" "oe:MOLEX_1719730004_1x04_P2.54mm_Vert_Lock"
 			(at 176.53 96.52 0)
 			(effects
